Commit message: Updated to allow for multi segment robot for machine learning algorithm

File: rceti_deployment/urdf/scene.urdf.xacro (robot description, xacro)
@@ -1,4 +1,5 @@
 <?xml version="1.0" ?>
 <robot name="scene" xmlns:xacro="http://ros.org/wiki/xacro">
+    <xacro:arg name="meshes_directory" default=""/>
     <!-- Setup -->
     <material name="environment_grey">

File: rceti_support/urdf/rceti_frame_macro.xacro (robot description, xacro)
@@ -169,36 +169,4 @@
             </visual>
         </link>
-        <link name="continuum_base_link_top">
-            <visual>
-                <geometry>
-                    <cylinder length="0.001" radius="0.001"/>
-                </geometry>
-                <origin xyz="0 0 0" rpy="0 0 0"/>
-            </visual>
-        </link>
-        <link name="continuum_base_link_bottom">
-            <visual>
-                <geometry>
-                    <cylinder length="0.001" radius="0.001"/>
-                </geometry>
-                <origin xyz="0 0 0" rpy="0 0 0"/>
-            </visual>
-        </link>
-        <link name="continuum_base_link_left">
-            <visual>
-                <geometry>
-                    <cylinder length="0.001" radius="0.001"/>
-                </geometry>
-                <origin xyz="0 0 0" rpy="0 0 0"/>
-            </visual>
-        </link>
-        <link name="continuum_base_link_right">
-            <visual>
-                <geometry>
-                    <cylinder length="0.001" radius="0.001"/>
-                </geometry>
-                <origin xyz="0 0 0" rpy="0 0 0"/>
-            </visual>
-        </link>
         <!-- JOINT GROUP -->
         <!-- Fixed Joint to ensure X actuator is anchored to the base link -->
@@ -244,32 +212,4 @@
             <origin xyz="0 0.017 0"/>
         </joint>
-        <joint name="continuum_top" type="revolute">
-            <parent link="pitch_servo_bottom_link"/>
-            <child link="continuum_base_link_top"/>
-            <origin xyz="0 0.017 0"/>
-            <axis xyz="0 0 1"/> <!-- Specify the axis of rotation -->
-            <limit effort="50.0" lower="-0.5" upper="0.5" velocity="1.0"/> <!-- Add limits -->
-        </joint>
-        <joint name="continuum_bottom" type="revolute">
-            <parent link="pitch_servo_bottom_link"/>
-            <child link="continuum_base_link_bottom"/>
-            <origin xyz="0 0.017 0"/>
-            <axis xyz="0 0 1"/> <!-- Specify the axis of rotation -->
-            <limit effort="50.0" lower="-0.5" upper="0.5" velocity="1.0"/> <!-- Add limits -->
-        </joint>
-        <joint name="continuum_left" type="revolute">
-            <parent link="pitch_servo_bottom_link"/>
-            <child link="continuum_base_link_left"/>
-            <origin xyz="0 0.017 0"/>
-            <axis xyz="0 0 1"/> <!-- Specify the axis of rotation -->
-            <limit effort="50.0" lower="-0.5" upper="0.5" velocity="1.0"/> <!-- Add limits -->
-        </joint>
-        <joint name="continuum_right" type="revolute">
-            <parent link="pitch_servo_bottom_link"/>
-            <child link="continuum_base_link_right"/>
-            <origin xyz="0 0.017 0"/>
-            <axis xyz="0 0 1"/> <!-- Specify the axis of rotation -->
-            <limit effort="50.0" lower="-0.5" upper="0.5" velocity="1.0"/> <!-- Add limits -->
-        </joint>
     </xacro:macro>
     <xacro:rceti_robot meshes_directory="$(arg meshes_directory)"/>
